File: smalAtmBoard.brd (EAGLE design)
At the start: 66.2 x 51.7 mm, 20 parts, among them IC1 ATMEGA-328P, IC2 7805-V, Y1 16MHz

Commit message: connector and routing
Parts:
- removed SV2: (no value), bauteile_jbt:FE03-2RAW
- added CON6: (no value), bauteile_jbt:FE05-2
- moved PAD22 6.84 mm to (41.0, 38.9)
- moved C5 1.65 mm to (56.5, 48.5)
- moved LED1 1.63 mm to (62.8, 48.1)
- moved C4 1.40 mm to (49.4, 48.5)
- moved IC2 1.02 mm to (15.2, 49.5)
- moved C101 0.97 mm to (61.2, 30.9), turned to 180 degrees
- moved S4 0.38 mm to (51.7, 4.95)
- moved R22 0.13 mm to (58.9, 12.4)
Connections:
- net AT-A0: now also CON6.3
- net AT-A4/SDA: now also CON6.7; no longer SV2.3
- net AT-A5/SCL: now also CON6.8; no longer SV2.4
- net AT-PD7: now also CON6.5
- net AT-PD8: now also CON6.6
- net GND: now also CON6.1, CON6.10; no longer SV2.1
- net VCC: now also CON6.2; no longer SV2.2
Routing:
- net RESET: track 0.00 -> 44.3 mm
- net VCC: track 0.00 -> 30.5 mm
- net TXD: track 0.00 -> 15.4 mm
- net RXD: track 0.00 -> 14.0 mm
- net AT-A4/SDA: track 0.00 -> 3.86 mm
- net AT-A3: track 0.00 -> 3.86 mm
- net AT-A2: track 0.00 -> 3.86 mm
- net AT-A1: track 0.00 -> 3.86 mm
- net AT-A0: track 0.00 -> 3.86 mm
- net AT-A5/SCL: track 0.00 -> 3.86 mm

Commit message: route
Parts:
- removed PAD22: D1, bauteile_jbt:PAD1,6/0,8
- added PAD1, PAD2, PAD3, PAD4, PAD5, PAD6: D1, bauteile_jbt:PAD1,6/0,8
- added SV2: (no value), con-lsta:FE08
- R16: value 1k -> 330
- moved R16 5.48 mm to (63.1, 48.5), turned to 0 degrees
- moved LED1 3.75 mm to (64.3, 44.7), turned to 90 degrees
- moved C2 1.36 mm to (61.4, 16.8), turned to 180 degrees
- moved R23 0.65 mm to (62.2, 12.3), turned to 90 degrees
- moved CON4 0.51 mm to (3.48, 21.3)
- moved Y1 0.25 mm to (59.3, 39.6)
- moved R22 0.18 mm to (58.8, 12.3), turned to 90 degrees
Connections:
- new net N$21: CON4.6, PAD1.1
- new net N$22: CON4.5, PAD2.1
- new net N$23: CON4.4, PAD3.1
- new net N$24: CON4.3, PAD4.1
- new net N$25: CON4.2, PAD5.1
- new net N$26: CON4.1, PAD6.1
- net AT-PD10: now also SV2.7; no longer PAD22.1
- net AT-PD11: now also SV2.6
- net AT-PD12: now also SV2.5
- net AT-PD2: now also SV2.1
- net AT-PD3: now also SV2.2
- net AT-PD4: now also SV2.3
- net AT-PD5: now also SV2.4
- net AT-PD9: now also SV2.8
Routing:
- net VCC: track 30.5 -> 93.1 mm
- net AT-PD8: track 0.00 -> 59.1 mm
- net AT-PD7: track 0.00 -> 52.4 mm
- net AT-PD13: track 0.00 -> 29.3 mm
- net AT-A5/SCL: track 3.86 -> 30.4 mm
- net AT-A0: track 3.86 -> 30.0 mm
- net AT-A4/SDA: track 3.86 -> 28.2 mm
- net XTAL2: track 0.00 -> 22.6 mm
- net XTAL1: track 0.00 -> 22.0 mm
- net AT-PD2: track 0.00 -> 16.9 mm
- net AT-PD4: track 0.00 -> 16.6 mm
- net AT-PD3: track 0.00 -> 16.6 mm
- net +12V: track 0.00 -> 14.2 mm
- net AT-PD5: track 0.00 -> 12.5 mm
- net AT-PD12: track 0.00 -> 3.78 mm
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
Commit message: finish routing
Parts:
- moved C5 2.03 mm to (54.5, 48.5)
- moved C4 1.91 mm to (47.5, 48.6)
- moved R16 1.28 mm to (61.8, 48.6)
- moved LED1 1.17 mm to (63.2, 45.0)
- moved IC2 1.17 mm to (14.5, 50.4)
- moved CON4 0.43 mm to (3.81, 21.5)
- moved PAD2 0.18 mm to (11.4, 24.1)
- moved PAD6 0.18 mm to (11.4, 3.81)
- moved PAD1 0.18 mm to (11.4, 29.2)
- moved PAD3 0.18 mm to (11.4, 19.1)
- moved PAD4 0.18 mm to (11.4, 14.0)
- moved PAD5 0.18 mm to (11.4, 8.89)
Connections:
- net VCC: now also CON6.9
Routing:
- net GND: track 0.00 -> 65.3 mm, vias 0 -> 12
- net VCC: track 93.1 -> 150.0 mm, vias 0 -> 10
- net N$26: track 0.00 -> 7.72 mm
- net N$25: track 0.00 -> 7.69 mm
- net N$21: track 0.00 -> 7.68 mm
- net N$22: track 0.00 -> 7.65 mm
- net N$24: track 0.00 -> 7.64 mm
- net N$23: track 0.00 -> 7.63 mm
- net XTAL2: track 22.6 -> 24.9 mm
- net XTAL1: track 22.0 -> 23.3 mm
- net AT-PD8: track 59.1 -> 57.8 mm
- net AT-PD7: track 52.4 -> 51.4 mm
- net AT-PD13: track 29.3 -> 28.3 mm
- net +12V: track 14.2 -> 13.5 mm
Other:
- board size 66.2 x 51.7 mm -> 66.1 x 51.7 mm
- board text added: "A0"
- board text added: "D12"
- board text added: "D5"
- board text added: "D7"
- board text added: "D8"
- board text added: "D9"
- board text added: "GND"
- board text added: "R"
- board text added: "RX"
- board text added: "SCL"
- board text added: "SDA"
- board text added: "TX"
- board text removed: "12"
- board text removed: "13"
- board text removed: "4"
- board text removed: "A1"
- board text removed: "A2"
- board text removed: "A3"
- board text removed: "A4"
- board text removed: "D0"
- board text removed: "D1"
- board text removed: "D4"
- board text removed: "~11"
- board text removed: "~D3"
- board text removed: "~D5"
- board text removed: "~D6"
