File: smalAtmBoard.sch (EAGLE design)
At the start: 18 parts, among them IC1 ATMEGA-328P, IC2 7805-V, Y1 16MHz

Commit message: connector and routing
Parts:
- removed SV2: (no value), bauteile_jbt:FE03-2FE03-2RAW
- added CON6: (no value), bauteile_jbt:FE05-2
Connections:
- net AT-A0: now also CON6.3
- net AT-A4/SDA: now also CON6.7; no longer SV2.3
- net AT-A5/SCL: now also CON6.8; no longer SV2.4
- net AT-PD7: now also CON6.5
- net AT-PD8: now also CON6.6
- net GND: now also CON6.1, CON6.10; no longer SV2.1
- net VCC: now also CON6.2; no longer SV2.2
Other:
- note added: "DISP / KBD / I2C"
Changed lines of the file:
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@@
 <?xml version="1.0" encoding="utf-8"?>
 <!DOCTYPE eagle SYSTEM "eagle.dtd">
-<eagle version="7.7.0">
+<eagle version="7.6.0">
 <drawing>
 <settings>
@@
 <part name="R22" library="bauteile_jbt" deviceset="R-EU_" device="0207/2V" value="2.2k"/>
 <part name="R23" library="bauteile_jbt" deviceset="R-EU_" device="0207/2V" value="2.2k"/>
-<part name="SV2" library="bauteile_jbt" deviceset="FE03-2" device="FE03-2RAW"/>
-<part name="GND24" library="supply1" deviceset="GND" device=""/>
-<part name="P+20" library="supply1" deviceset="VCC" device="" value="VCC"/>
 <part name="P+23" library="supply1" deviceset="VCC" device="" value="VCC"/>
 <part name="P+24" library="supply1" deviceset="VCC" device="" value="VCC"/>
 <part name="SV3" library="con-lsta" deviceset="FE06-1" device=""/>
+<part name="CON6" library="bauteile_jbt" deviceset="FE05-2" device=""/>
+<part name="P+3" library="supply1" deviceset="VCC" device=""/>
+<part name="GND5" library="supply1" deviceset="GND" device=""/>
+<part name="GND6" library="supply1" deviceset="GND" device=""/>
 </parts>
 <sheets>
@@
 <text x="218.44" y="40.64" size="1.778" layer="91">Serial Connector</text>
 <text x="252.222" y="215.9" size="2.54" layer="91">12V Supply</text>
-<text x="170.18" y="220.98" size="1.778" layer="91">I2C interface</text>
+<text x="160.02" y="208.28" size="1.778" layer="91">I2C interface</text>
+<text x="269.24" y="132.08" size="5.08" layer="91">DISP / KBD / I2C</text>
 </plain>
 <instances>
@@
 <instance part="R22" gate="G$1" x="190.5" y="185.42" rot="R270"/>
 <instance part="R23" gate="G$1" x="160.02" y="185.42" rot="R270"/>
-<instance part="SV2" gate="G$1" x="175.26" y="200.66" rot="R180"/>
-<instance part="GND24" gate="1" x="195.58" y="213.36" rot="R180"/>
-<instance part="P+20" gate="VCC" x="152.4" y="220.98" smashed="yes">
-<attribute name="VALUE" x="154.305" y="223.52" size="1.778" layer="96" rot="R180"/>
-</instance>
 <instance part="P+23" gate="VCC" x="147.32" y="185.42" smashed="yes">
 <attribute name="VALUE" x="149.225" y="187.96" size="1.778" layer="96" rot="R180"/>
@@
 </instance>
 <instance part="SV3" gate="G$1" x="152.4" y="134.62" rot="R270"/>
+<instance part="CON6" gate="G$1" x="325.12" y="96.52" rot="R90"/>
+<instance part="P+3" gate="VCC" x="330.2" y="124.46" smashed="yes">
+<attribute name="VALUE" x="332.105" y="127" size="1.778" layer="96" rot="R180"/>
+</instance>
+<instance part="GND5" gate="1" x="345.44" y="81.28"/>
+<instance part="GND6" gate="1" x="299.72" y="93.98"/>
 </instances>
 <busses>
@@
 </segment>
 <segment>
-<pinref part="GND24" gate="1" pin="GND"/>
-<pinref part="SV2" gate="G$1" pin="1"/>
-<wire x1="195.58" y1="210.82" x2="195.58" y2="203.2" width="0.1524" layer="91"/>
-<wire x1="195.58" y1="203.2" x2="182.88" y2="203.2" width="0.1524" layer="91"/>
+<pinref part="GND5" gate="1" pin="GND"/>
+<pinref part="CON6" gate="G$1" pin="1"/>
+<wire x1="345.44" y1="83.82" x2="330.2" y2="83.82" width="0.1524" layer="91"/>
+<wire x1="330.2" y1="83.82" x2="330.2" y2="88.9" width="0.1524" layer="91"/>
+</segment>
+<segment>
+<pinref part="CON6" gate="G$1" pin="10"/>
+<pinref part="GND6" gate="1" pin="GND"/>
+<wire x1="320.04" y1="104.14" x2="299.72" y2="104.14" width="0.1524" layer="91"/>
+<wire x1="299.72" y1="104.14" x2="299.72" y2="96.52" width="0.1524" layer="91"/>
 </segment>
 </net>
@@
 </segment>
 <segment>
-<pinref part="P+20" gate="VCC" pin="VCC"/>
-<pinref part="SV2" gate="G$1" pin="2"/>
-<wire x1="152.4" y1="218.44" x2="152.4" y2="203.2" width="0.1524" layer="91"/>
-<wire x1="152.4" y1="203.2" x2="167.64" y2="203.2" width="0.1524" layer="91"/>
-</segment>
-<segment>
 <pinref part="R23" gate="G$1" pin="2"/>
 <wire x1="160.02" y1="175.26" x2="160.02" y2="180.34" width="0.1524" layer="91"/>
@@
 <pinref part="P+24" gate="VCC" pin="VCC"/>
 <wire x1="200.66" y1="175.26" x2="200.66" y2="182.88" width="0.1524" layer="91"/>
+</segment>
+<segment>
+<pinref part="P+3" gate="VCC" pin="VCC"/>
+<pinref part="CON6" gate="G$1" pin="2"/>
+<wire x1="330.2" y1="121.92" x2="330.2" y2="104.14" width="0.1524" layer="91"/>
 </segment>
 </net>
@@
 <label x="137.16" y="53.34" size="1.778" layer="95"/>
 </segment>
+<segment>
+<wire x1="266.7" y1="73.66" x2="325.12" y2="73.66" width="0.1524" layer="91"/>
+<label x="304.8" y="73.66" size="1.778" layer="95"/>
+<pinref part="CON6" gate="G$1" pin="5"/>
+<wire x1="325.12" y1="73.66" x2="325.12" y2="88.9" width="0.1524" layer="91"/>
+</segment>
 </net>
 <net name="AT-A4/SDA" class="0">
@@
 </segment>
 <segment>
-<pinref part="SV2" gate="G$1" pin="3"/>
 <wire x1="205.74" y1="200.66" x2="190.5" y2="200.66" width="0.1524" layer="91"/>
 <wire x1="190.5" y1="200.66" x2="182.88" y2="200.66" width="0.1524" layer="91"/>
@@
 <wire x1="190.5" y1="190.5" x2="190.5" y2="200.66" width="0.1524" layer="91"/>
 <label x="195.58" y="200.66" size="1.778" layer="95"/>
+</segment>
+<segment>
+<label x="304.8" y="78.74" size="1.778" layer="95"/>
+<wire x1="322.58" y1="78.74" x2="304.8" y2="78.74" width="0.1524" layer="91"/>
+<pinref part="CON6" gate="G$1" pin="7"/>
+<wire x1="322.58" y1="78.74" x2="322.58" y2="88.9" width="0.1524" layer="91"/>
 </segment>
 </net>
@@
 <label x="137.16" y="50.8" size="1.778" layer="95"/>
 </segment>
+<segment>
+<wire x1="325.12" y1="111.76" x2="266.7" y2="111.76" width="0.1524" layer="91"/>
+<label x="294.64" y="111.76" size="1.778" layer="95"/>
+<pinref part="CON6" gate="G$1" pin="6"/>
+<wire x1="325.12" y1="111.76" x2="325.12" y2="104.14" width="0.1524" layer="91"/>
+</segment>
 </net>
 <net name="AT-PD9" class="0">
@@
 <wire x1="167.64" y1="200.66" x2="160.02" y2="200.66" width="0.1524" layer="91"/>
 <label x="144.78" y="200.66" size="1.778" layer="95"/>
-<pinref part="SV2" gate="G$1" pin="4"/>
 <wire x1="160.02" y1="200.66" x2="142.24" y2="200.66" width="0.1524" layer="91"/>
 <wire x1="160.02" y1="190.5" x2="160.02" y2="200.66" width="0.1524" layer="91"/>
 <junction x="160.02" y="200.66"/>
+</segment>
+<segment>
+<label x="302.26" y="106.68" size="1.778" layer="95"/>
+<wire x1="322.58" y1="106.68" x2="302.26" y2="106.68" width="0.1524" layer="91"/>
+<pinref part="CON6" gate="G$1" pin="8"/>
+<wire x1="322.58" y1="106.68" x2="322.58" y2="104.14" width="0.1524" layer="91"/>
 </segment>
 </net>
@@
 <wire x1="147.32" y1="127" x2="147.32" y2="93.98" width="0.1524" layer="91"/>
 </segment>
-</net>
+<segment>
+<wire x1="327.66" y1="58.42" x2="312.42" y2="58.42" width="0.1524" layer="91"/>
+<label x="314.96" y="58.42" size="1.778" layer="95"/>
+<pinref part="CON6" gate="G$1" pin="3"/>
+<wire x1="327.66" y1="58.42" x2="327.66" y2="88.9" width="0.1524" layer="91"/>
+</segment>
+</net>

Commit message: route
Parts:
- removed PAD22: D1, bauteile_jbt:PAD1,6/0,8
- added PAD1, PAD2, PAD3, PAD4, PAD5, PAD6: D1, bauteile_jbt:PAD1,6/0,8
- added SV2: (no value), con-lsta:FE08-1
- R16: value 1k -> 330
Connections:
- new net N$21: CON4-6.KL, PAD1.P
- new net N$22: CON4-5.KL, PAD2.P
- new net N$23: CON4-4.KL, PAD3.P
- new net N$24: CON4-3.KL, PAD4.P
- new net N$25: CON4-2.KL, PAD5.P
- new net N$26: CON4-1.KL, PAD6.P
- net AT-PD10: now also SV2.7; no longer PAD22.P
- net AT-PD11: now also SV2.6
- net AT-PD12: now also SV2.5
- net AT-PD2: now also SV2.1
- net AT-PD3: now also SV2.2
- net AT-PD4: now also SV2.3
- net AT-PD5: now also SV2.4
- net AT-PD9: now also SV2.8
Other:
- note added: "I2C interface^pullups"
- note removed: "I2C interface"
- moved on the sheet: IC2, LED1, R16, R22, R23, SV1

Commit message: finish routing
Connections:
- net VCC: now also CON6.9
Changed lines of the file:
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@@
 <grid distance="0.1" unitdist="inch" unit="inch" style="lines" multiple="1" display="no" altdistance="0.01" altunitdist="inch" altunit="inch"/>
 <layers>
-<layer number="1" name="Top" color="4" fill="1" visible="no" active="no"/>
-<layer number="2" name="Route2" color="1" fill="3" visible="no" active="no"/>
-<layer number="3" name="Route3" color="4" fill="3" visible="no" active="no"/>
-<layer number="14" name="Route14" color="1" fill="6" visible="no" active="no"/>
-<layer number="15" name="Route15" color="4" fill="6" visible="no" active="no"/>
-<layer number="16" name="Bottom" color="1" fill="1" visible="no" active="no"/>
-<layer number="17" name="Pads" color="2" fill="1" visible="no" active="no"/>
-<layer number="18" name="Vias" color="14" fill="1" visible="no" active="no"/>
-<layer number="19" name="Unrouted" color="6" fill="1" visible="no" active="no"/>
-<layer number="20" name="Dimension" color="15" fill="1" visible="no" active="no"/>
-<layer number="21" name="tPlace" color="7" fill="1" visible="no" active="no"/>
-<layer number="22" name="bPlace" color="7" fill="1" visible="no" active="no"/>
-<layer number="23" name="tOrigins" color="15" fill="1" visible="no" active="no"/>
-<layer number="24" name="bOrigins" color="15" fill="1" visible="no" active="no"/>
-<layer number="25" name="tNames" color="7" fill="1" visible="no" active="no"/>
-<layer number="26" name="bNames" color="7" fill="1" visible="no" active="no"/>
-<layer number="27" name="tValues" color="7" fill="1" visible="no" active="no"/>
-<layer number="28" name="bValues" color="7" fill="1" visible="no" active="no"/>
+<layer number="1" name="Top" color="4" fill="1" visible="yes" active="no"/>
+<layer number="2" name="Route2" color="1" fill="3" visible="yes" active="no"/>
+<layer number="3" name="Route3" color="4" fill="3" visible="yes" active="no"/>
+<layer number="14" name="Route14" color="1" fill="6" visible="yes" active="no"/>
+<layer number="15" name="Route15" color="4" fill="6" visible="yes" active="no"/>
+<layer number="16" name="Bottom" color="1" fill="1" visible="yes" active="no"/>
+<layer number="17" name="Pads" color="2" fill="1" visible="yes" active="no"/>
+<layer number="18" name="Vias" color="14" fill="1" visible="yes" active="no"/>
+<layer number="19" name="Unrouted" color="6" fill="1" visible="yes" active="no"/>
+<layer number="20" name="Dimension" color="15" fill="1" visible="yes" active="no"/>
+<layer number="21" name="tPlace" color="7" fill="1" visible="yes" active="no"/>
+<layer number="22" name="bPlace" color="7" fill="1" visible="yes" active="no"/>
+<layer number="23" name="tOrigins" color="15" fill="1" visible="yes" active="no"/>
+<layer number="24" name="bOrigins" color="15" fill="1" visible="yes" active="no"/>
+<layer number="25" name="tNames" color="7" fill="1" visible="yes" active="no"/>
+<layer number="26" name="bNames" color="7" fill="1" visible="yes" active="no"/>
+<layer number="27" name="tValues" color="7" fill="1" visible="yes" active="no"/>
+<layer number="28" name="bValues" color="7" fill="1" visible="yes" active="no"/>
 <layer number="29" name="tStop" color="7" fill="3" visible="no" active="no"/>
 <layer number="30" name="bStop" color="7" fill="6" visible="no" active="no"/>
@@
 <layer number="35" name="tGlue" color="7" fill="4" visible="no" active="no"/>
 <layer number="36" name="bGlue" color="7" fill="5" visible="no" active="no"/>
-<layer number="37" name="tTest" color="7" fill="1" visible="no" active="no"/>
-<layer number="38" name="bTest" color="7" fill="1" visible="no" active="no"/>
+<layer number="37" name="tTest" color="7" fill="1" visible="yes" active="no"/>
+<layer number="38" name="bTest" color="7" fill="1" visible="yes" active="no"/>
 <layer number="39" name="tKeepout" color="4" fill="11" visible="no" active="no"/>
 <layer number="40" name="bKeepout" color="1" fill="11" visible="no" active="no"/>
@@
 <layer number="44" name="Drills" color="7" fill="1" visible="no" active="no"/>
 <layer number="45" name="Holes" color="7" fill="1" visible="no" active="no"/>
-<layer number="46" name="Milling" color="3" fill="1" visible="no" active="no"/>
-<layer number="47" name="Measures" color="7" fill="1" visible="no" active="no"/>
-<layer number="48" name="Document" color="7" fill="1" visible="no" active="no"/>
-<layer number="49" name="Reference" color="7" fill="1" visible="no" active="no"/>
-<layer number="50" name="dxf" color="12" fill="1" visible="no" active="no"/>
-<layer number="51" name="tDocu" color="7" fill="1" visible="no" active="no"/>
-<layer number="52" name="bDocu" color="7" fill="1" visible="no" active="no"/>
+<layer number="46" name="Milling" color="3" fill="1" visible="yes" active="no"/>
+<layer number="47" name="Measures" color="7" fill="1" visible="yes" active="no"/>
+<layer number="48" name="Document" color="7" fill="1" visible="yes" active="no"/>
+<layer number="49" name="Reference" color="7" fill="1" visible="yes" active="no"/>
+<layer number="50" name="dxf" color="12" fill="1" visible="yes" active="no"/>
+<layer number="51" name="tDocu" color="7" fill="1" visible="yes" active="no"/>
+<layer number="52" name="bDocu" color="7" fill="1" visible="yes" active="no"/>
 <layer number="91" name="Nets" color="2" fill="1" visible="yes" active="yes"/>
 <layer number="92" name="Busses" color="1" fill="1" visible="yes" active="yes"/>
@@
 <layer number="95" name="Names" color="7" fill="1" visible="yes" active="yes"/>
 <layer number="96" name="Values" color="7" fill="1" visible="yes" active="yes"/>
-<layer number="53" name="tGND_GNDA" color="7" fill="1" visible="no" active="no"/>
-<layer number="54" name="bGND_GNDA" color="7" fill="1" visible="no" active="no"/>
-<layer number="56" name="wert" color="7" fill="1" visible="no" active="no"/>
-<layer number="57" name="tCAD" color="7" fill="1" visible="no" active="no"/>
-<layer number="59" name="tCarbon" color="7" fill="1" visible="no" active="no"/>
-<layer number="60" name="bCarbon" color="7" fill="1" visible="no" active="no"/>
+<layer number="53" name="tGND_GNDA" color="7" fill="1" visible="yes" active="no"/>
+<layer number="54" name="bGND_GNDA" color="7" fill="1" visible="yes" active="no"/>
+<layer number="56" name="wert" color="7" fill="1" visible="yes" active="no"/>
+<layer number="57" name="tCAD" color="7" fill="1" visible="yes" active="no"/>
+<layer number="59" name="tCarbon" color="7" fill="1" visible="yes" active="no"/>
+<layer number="60" name="bCarbon" color="7" fill="1" visible="yes" active="no"/>
 <layer number="90" name="Modules" color="5" fill="1" visible="no" active="no"/>
 <layer number="97" name="Info" color="7" fill="1" visible="no" active="no"/>
@@
 <pinref part="P+3" gate="VCC" pin="VCC"/>
 <pinref part="CON6" gate="G$1" pin="2"/>
-<wire x1="330.2" y1="121.92" x2="330.2" y2="104.14" width="0.1524" layer="91"/>
+<wire x1="330.2" y1="121.92" x2="330.2" y2="109.22" width="0.1524" layer="91"/>
+<pinref part="CON6" gate="G$1" pin="9"/>
+<wire x1="330.2" y1="109.22" x2="330.2" y2="104.14" width="0.1524" layer="91"/>
+<wire x1="320.04" y1="88.9" x2="320.04" y2="86.36" width="0.1524" layer="91"/>
+<wire x1="320.04" y1="86.36" x2="335.28" y2="86.36" width="0.1524" layer="91"/>
+<wire x1="335.28" y1="86.36" x2="335.28" y2="109.22" width="0.1524" layer="91"/>
+<wire x1="335.28" y1="109.22" x2="330.2" y2="109.22" width="0.1524" layer="91"/>
+<junction x="330.2" y="109.22"/>
 </segment>
 </net>
