File: smallAtmBoard.sch (EAGLE design)
At the start: 24 parts, among them IC1 ATMEGA-328P, IC2 7805-V, Y1 16MHz

Commit message: new connectors + routing
Parts:
- added U$2: FE02-2, bauteile_jbt:FE02-2
- CON6: device bauteile_jbt:FE05-2 -> bauteile_jbt:FE03-2
- SV2: device con-lsta:FE08-1 -> bauteile_jbt:FE08-1
Connections:
- net AT-A4/SDA: now also U$2.3; no longer CON6.7
- net AT-A5/SCL: now also U$2.4; no longer CON6.8
- net AT-PD6: now also CON6.4
- net GND: now also U$2.1; no longer CON6.10
- net VCC: now also U$2.2; no longer CON6.9
Other:
- note added: "5V Supply"
- note added: "Connector for Display / Keyboard"
- note added: "Connector for I2C"
- note added: "Controller with Connector for LCD"
- note removed: "12V Supply"
- note removed: "Controller / LCD / Latch / RTC"
- note removed: "DISP / KBD / I2C"
- note removed: "I2C interface^pullups"
- moved on the sheet: C101, C2, C4, C5, IC1, LED1, R16, R22, R23, R3, S4, SV1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
